File: Projekt UE.kicad_pcb (KiCad board)
At the start: 2 copper layers, 67 parts, among them J1 NEB_21_R, J2 502382-0670, J3 TB006-508-12BE, J4 1935187, J5 215297-8, K1 V23061B1007A301, K2 V23061B1007A301, K3 V23061B1007A301, K4 V23061B1007A301, K5 V23061B1007A301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

Commit message: Upload pcb after load footprint
Connections:
- U4 pad 17: unconnected-(U4-Pad17) -> +3.3V
